File: Hardware/PCB/pcbdraft-2/pcbdraft-2.kicad_pcb (KiCad board)
At the start: 2 copper layers, 17 parts, among them J1 RJ45, J10 RJ45, J11 RJ45, J12 RJ45, J13 RJ45, J14 RJ45, J15 RJ45, J16 RJ45, J2 RJ45, J3 RJ45, J4 RJ45, J5 RJ45, J6 RJ45, J7 RJ45, J8 RJ45, J9 RJ45

Commit message: updated redesigned board
Parts:
- added G***: LOGO, LOGO, F.Cu at (99.1, 137.7)
- added J17: Enable, Connector_PinHeader_2.54mm:PinHeader_1x02_P2.54mm_Vertical, F.Cu at (183.9, 78.2)
- added R1: R, Resistor_SMD:R_0805_2012Metric_Pad1.20x1.40mm_HandSolder, F.Cu at (155.0, 85.9)
- added R2: R, Resistor_SMD:R_0805_2012Metric_Pad1.20x1.40mm_HandSolder, F.Cu at (155.0, 88.4)
- added R3: R, Resistor_SMD:R_0805_2012Metric_Pad1.20x1.40mm_HandSolder, F.Cu at (155.0, 90.9)
- added R4: R, Resistor_SMD:R_0805_2012Metric_Pad1.20x1.40mm_HandSolder, F.Cu at (155.0, 96.0)
- added R5: R, Resistor_SMD:R_0805_2012Metric_Pad1.20x1.40mm_HandSolder, F.Cu at (155.0, 98.6)
- added R6: R, Resistor_SMD:R_0805_2012Metric_Pad1.20x1.40mm_HandSolder, F.Cu at (155.0, 101.1)
- added R7: R, Resistor_SMD:R_0805_2012Metric_Pad1.20x1.40mm_HandSolder, F.Cu at (155.0, 103.6)
- added R8: R, Resistor_SMD:R_0805_2012Metric_Pad1.20x1.40mm_HandSolder, F.Cu at (155.0, 106.2)
- moved A1 42.5 mm to (159.0, 68.1)
- moved J11 11.9 mm to (116.8, 94.0)
- moved J12 11.9 mm to (134.6, 94.0)
- moved J15 11.9 mm to (116.8, 112.5)
- moved J16 11.9 mm to (134.6, 112.5)
- moved J7 11.5 mm to (116.8, 73.0)
- moved J8 11.5 mm to (134.6, 73.0)
- moved J3 11.5 mm to (116.8, 54.5)
- moved J4 11.5 mm to (134.6, 54.5)
- moved J13 10.9 mm to (80.3, 112.5)
- moved J9 10.9 mm to (80.3, 94.0)
- moved J14 10.9 mm to (98.0, 112.5)
- moved J10 10.9 mm to (98.0, 94.0)
- moved J1 10.4 mm to (80.3, 54.5)
- moved J5 10.4 mm to (80.3, 73.0)
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Connections:
- A1 pad 10: C2 -> Net-(A1-A5)
- A1 pad 11: C3 -> unconnected-(A1-SCK-Pad11)
- A1 pad 12: C1 -> Net-(A1-MOSI)
- A1 pad 13: R1 -> Net-(A1-MISO)
- A1 pad 14: R3 -> Net-(A1-RX)
- A1 pad 15: R5 -> Net-(A1-TX)
- A1 pad 16: unconnected-(A1-SPARE-Pad16) -> Net-(A1-SPARE)
- A1 pad 17: R7 -> unconnected-(A1-SDA-Pad17)
- A1 pad 18: C8 -> R8
- A1 pad 19: C6 -> R6
- A1 pad 20: C7 -> R4
- A1 pad 21: C5 -> R2
- A1 pad 22: unconnected-(A1-D3-Pad22) -> R7
- A1 pad 23: unconnected-(A1-D4-Pad23) -> R5
- A1 pad 24: unconnected-(A1-D5-Pad24) -> R3
- A1 pad 25: unconnected-(A1-D6-Pad25) -> R1
- A1 pad 27: unconnected-(A1-EN-Pad27) -> Net-(A1-EN)
- A1 pad 4: unconnected-(A1-GND-Pad4) -> GND
- A1 pad 5: R2 -> unconnected-(A1-A0-Pad5)
- A1 pad 6: R4 -> unconnected-(A1-A1-Pad6)
- A1 pad 7: R6 -> unconnected-(A1-A2-Pad7)
- A1 pad 8: R8 -> Net-(A1-A3)
- A1 pad 9: C4 -> Net-(A1-A4)
- J10 pad 1: R6 -> R5
- J10 pad 2: C1 -> C5
- J10 pad 3: R6 -> R5
- J10 pad 4: C2 -> C6
- J10 pad 5: R6 -> R5
- J10 pad 6: C3 -> C7
- J10 pad 7: R6 -> R5
- J10 pad 8: C4 -> C8
- J11 pad 1: R7 -> R6
- J11 pad 3: R7 -> R6
- J11 pad 5: R7 -> R6
- J11 pad 7: R7 -> R6
- J12 pad 1: R8 -> R6
- J12 pad 2: C1 -> C5
- J12 pad 3: R8 -> R6
- J12 pad 4: C2 -> C6
- J12 pad 5: R8 -> R6
- J12 pad 6: C3 -> C7
- J12 pad 7: R8 -> R6
- J12 pad 8: C4 -> C8
- J13 pad 1: R5 -> R7
- J13 pad 2: C5 -> C1
- J13 pad 3: R5 -> R7
- J13 pad 4: C6 -> C2
- J13 pad 5: R5 -> R7
- J13 pad 6: C7 -> C3
- J13 pad 7: R5 -> R7
- J13 pad 8: C8 -> C4
- J14 pad 1: R6 -> R7
- J14 pad 3: R6 -> R7
- J14 pad 5: R6 -> R7
- J14 pad 7: R6 -> R7
- J15 pad 1: R7 -> R8
- J15 pad 2: C5 -> C1
- J15 pad 3: R7 -> R8
- J15 pad 4: C6 -> C2
- J15 pad 5: R7 -> R8
- J15 pad 6: C7 -> C3
- J15 pad 7: R7 -> R8
- J15 pad 8: C8 -> C4
Routing:
- net R1: track 0.00 -> 261.4 mm
- net C4: track 0.00 -> 245.2 mm, vias 0 -> 1
- net R3: track 0.00 -> 238.2 mm
- net C1: track 0.00 -> 229.8 mm
- net C2: track 0.00 -> 228.2 mm, vias 0 -> 1
- net C3: track 0.00 -> 226.1 mm
- net R5: track 0.00 -> 212.3 mm
- net R2: track 0.00 -> 208.0 mm
- net C8: track 0.00 -> 196.9 mm, vias 0 -> 1
- net R7: track 0.00 -> 188.4 mm
- net C6: track 0.00 -> 184.7 mm
- net R4: track 0.00 -> 184.6 mm
- net C5: track 0.00 -> 184.4 mm
- net C7: track 0.00 -> 183.2 mm, vias 0 -> 1
- net R6: track 0.00 -> 159.4 mm
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Other:
- board outline added: 115.3 x 101.6 mm
- board text added: "5/17/2024"
- board text added: "Arduino Component Storage Cart Rev 2.0"
- board text added: "Cat5E Twisted Pair Pinout #--------------# Pins 1-2 -- LED 1 Pins 3-4 -- LED 2 Pins 5-6 -- LED 3 Pins 7-8 -- LED 4"
- board text added: "Designed By: Michael B. Lance"
- board text removed: "2/5/2024"

Commit message: minor revisions
Other:
- board text added: "2.0"
- board text removed: "1.0"
Changed lines of the file:
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@@
 		)
 	)
-	(gr_text "1.0\n"
+	(gr_text "2.0\n"
 		(at 268.224 194.056 0)
 		(layer "F.Cu")
